File: SipPuffDuoOutputs/SipPuffDuoOutputsATtiny84MOSFET/SipPuffDuoOutputsATtiny84MOSFET.sch (EAGLE design)
At the start: 19 parts, among them U1 ATTINY84-20PU, U2 4936BM08A-M, U3 4936BM08A-M

Commit message: Changed resistors size
Parts:
- R1: device MMC Eagle:RESISTOR_R-US_0204/5 -> MMC Eagle:RESISTOR_R-US_
Changed lines of the file:
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@@
 <part name="U3" library="MMC Eagle" library_urn="urn:adsk.eagle:library:3491419" deviceset="4936B" device="M08A-M" package3d_urn="urn:adsk.eagle:package:4704332/2"/>
 <part name="D1" library="MMC Eagle" library_urn="urn:adsk.eagle:library:3491419" deviceset="LED" device="5MM" package3d_urn="urn:adsk.eagle:package:3634149/2"/>
-<part name="R1" library="MMC Eagle" library_urn="urn:adsk.eagle:library:3491419" deviceset="RESISTOR_R-US_" device="0204/5" package3d_urn="urn:adsk.eagle:package:3491543/2" value="1k"/>
+<part name="R1" library="MMC Eagle" library_urn="urn:adsk.eagle:library:3491419" deviceset="RESISTOR_R-US_" device="" package3d_urn="urn:adsk.eagle:package:5426338/2" value="1k"/>
 <part name="GND6" library="MMC Eagle" library_urn="urn:adsk.eagle:library:3491419" deviceset="GND" device=""/>
 <part name="U$1" library="MMC Eagle" library_urn="urn:adsk.eagle:library:3491419" deviceset="HEADER_2X03" device="" package3d_urn="urn:adsk.eagle:package:4704386/2"/>
