File: SipPuffOneOutput/SipPuffOneOuputATtiny85MOSFET/SipPuffOneOuputATtiny85MOSFET.sch (EAGLE design)
At the start: 13 parts, among them U1 ATTINY85-20PU, U2 4936BM08A-M

Commit message: Changed resistors size
Parts:
- R1: device MMC Eagle:RESISTOR_R-US_0204/7 -> MMC Eagle:RESISTOR_R-US_
Changed lines of the file:
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@@
 <part name="C2" library="MMC Eagle" library_urn="urn:adsk.eagle:library:3491419" deviceset="0.1UF" device="-KIT-EZ-50V-20%" package3d_urn="urn:adsk.eagle:package:3493607/2" value="0.01uF"/>
 <part name="C3" library="MMC Eagle" library_urn="urn:adsk.eagle:library:3491419" deviceset="0.1UF" device="-KIT-EZ-50V-20%" package3d_urn="urn:adsk.eagle:package:3493607/2" value="1uF"/>
-<part name="R1" library="MMC Eagle" library_urn="urn:adsk.eagle:library:3491419" deviceset="RESISTOR_R-US_" device="0204/7" package3d_urn="urn:adsk.eagle:package:3491542/2"/>
+<part name="R1" library="MMC Eagle" library_urn="urn:adsk.eagle:library:3491419" deviceset="RESISTOR_R-US_" device="" package3d_urn="urn:adsk.eagle:package:5426338/2"/>
 <part name="D1" library="MMC Eagle" library_urn="urn:adsk.eagle:library:3491419" deviceset="LED" device="5MM" package3d_urn="urn:adsk.eagle:package:3634149/2"/>
 <part name="GND1" library="MMC Eagle" library_urn="urn:adsk.eagle:library:3491419" deviceset="GND" device=""/>
