File: SipPuffOneOutput/SipPuffOneOuputATtiny85Relay/SipPuffOneOuputATtiny85Relays.brd (EAGLE design)
At the start: 48 x 70 mm, 13 parts, among them U1 ATTINY85-20PU, U2 AQY212EH

Commit message: Changed resistors size
Parts:
- added R2: 2k, MMC Eagle:RESISTOR_0207/10
- added R3: 1k, MMC Eagle:RESISTOR_0207/10
- R1: device MMC Eagle:RESISTOR_0204/7 -> MMC Eagle:RESISTOR_0207/10
Connections:
- new net N$11: R2.2, R3.1
- new net N$14: R3.2, U2.1
- net N$6: now also R2.1; no longer U2.1
Routing:
- net N$14: track 0.00 -> 4.56 mm
- net N$11: track 0.00 -> 3.00 mm
- net N$5: track 8.17 -> 6.90 mm
- net N$4: track 6.89 -> 5.62 mm
- net N$6: track 46.5 -> 45.7 mm
Changed lines of the file:
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@@
 <drawing>
 <settings>
-<setting alwaysvectorfont="yes"/>
+<setting alwaysvectorfont="no"/>
 <setting verticaltext="up"/>
 </settings>
@@
 <attribute name="VALUE" x="20.444" y="14.89" size="1.27" layer="27"/>
 </element>
-<element name="R1" library="MMC Eagle" library_urn="urn:adsk.eagle:library:3491419" package="RESISTOR_0204/7" package3d_urn="urn:adsk.eagle:package:3491542/2" value="" x="22.73" y="38.02" smashed="yes" rot="R270">
+<element name="R1" library="MMC Eagle" library_urn="urn:adsk.eagle:library:3491419" package="RESISTOR_0207/10" package3d_urn="urn:adsk.eagle:package:5426338/2" value="" x="22.73" y="38.02" smashed="yes" rot="R270">
 <attribute name="VALUE" x="22.2474" y="39.6456" size="0.9906" layer="27" ratio="10" rot="R270"/>
 </element>
@@
 <element name="U$4" library="MMC Eagle" library_urn="urn:adsk.eagle:library:3491419" package="2X3" package3d_urn="urn:adsk.eagle:package:4704386/2" value="HEADER_2X03" x="7" y="24" smashed="yes" rot="R270"/>
 <element name="U$5" library="MMC Eagle" library_urn="urn:adsk.eagle:library:3491419" package="1X02" package3d_urn="urn:adsk.eagle:package:4737896/2" value="HEADER_1X02" x="7" y="15" smashed="yes"/>
+<element name="R2" library="MMC Eagle" library_urn="urn:adsk.eagle:library:3491419" package="RESISTOR_0207/10" package3d_urn="urn:adsk.eagle:package:5426338/2" value="2k" x="40.5" y="36.5" smashed="yes" rot="R270">
+<attribute name="VALUE" x="41.865" y="37.2606" size="1.27" layer="27" ratio="10" rot="R270"/>
+</element>
+<element name="R3" library="MMC Eagle" library_urn="urn:adsk.eagle:library:3491419" package="RESISTOR_0207/10" package3d_urn="urn:adsk.eagle:package:5426338/2" value="1k" x="37.5" y="36.5" smashed="yes" rot="R90">
+<attribute name="VALUE" x="36.135" y="35.7394" size="1.27" layer="27" ratio="10" rot="R90"/>
+</element>
 </elements>
 <signals>
@@
 <contactref element="U1" pad="3"/>
 <contactref element="R1" pad="2"/>
-<wire x1="22.73" y1="34.21" x2="22.73" y2="27.63" width="0.1524" layer="1"/>
+<wire x1="22.73" y1="32.94" x2="22.73" y2="27.63" width="0.1524" layer="1"/>
 <wire x1="22.73" y1="27.63" x2="22.95" y2="27.41" width="0.1524" layer="1"/>
 </signal>
@@
 <contactref element="R1" pad="1"/>
 <contactref element="D1" pad="A"/>
-<wire x1="22.73" y1="50" x2="22.73" y2="41.83" width="0.1524" layer="1"/>
+<wire x1="22.73" y1="50" x2="22.73" y2="43.1" width="0.1524" layer="1"/>
 </signal>
 <signal name="GND">
@@
 <vertex x="-2.5" y="-2"/>
 </polygon>
+<contactref element="U$4" pad="3"/>
 <contactref element="U2" pad="2"/>
-<contactref element="U$4" pad="3"/>
 </signal>
 <signal name="N$3">
@@
 <signal name="N$6">
 <contactref element="U1" pad="7"/>
-<contactref element="U2" pad="1"/>
 <contactref element="U$4" pad="2"/>
-<wire x1="25.49" y1="19.79" x2="34.46" y2="28.76" width="0.1524" layer="1"/>
-<wire x1="34.46" y1="28.76" x2="34.46" y2="44.88" width="0.1524" layer="1"/>
 <wire x1="21.28" y1="24" x2="25.49" y2="19.79" width="0.1524" layer="1"/>
 <wire x1="9.54" y1="24" x2="21.28" y2="24" width="0.1524" layer="1"/>
+<contactref element="R2" pad="1"/>
+<wire x1="25.49" y1="19.79" x2="31.5" y2="25.8" width="0.1524" layer="1"/>
+<wire x1="31.5" y1="25.8" x2="31.5" y2="29.5" width="0.1524" layer="1"/>
+<wire x1="31.5" y1="29.5" x2="40.5" y2="38.5" width="0.1524" layer="1"/>
+<wire x1="40.5" y1="38.5" x2="40.5" y2="41.58" width="0.1524" layer="1"/>
 </signal>
 <signal name="N$7">
@@
 <wire x1="19.5" y1="24" x2="22.08" y2="24" width="0.1524" layer="16"/>
 </signal>
+<signal name="N$11">
+<contactref element="R2" pad="2"/>
+<contactref element="R3" pad="1"/>
+<wire x1="37.5" y1="31.42" x2="40.5" y2="31.42" width="0.1524" layer="1"/>
+</signal>
+<signal name="N$14">
+<contactref element="R3" pad="2"/>
+<contactref element="U2" pad="1"/>
+<wire x1="34.46" y1="44.88" x2="37.5" y2="41.84" width="0.1524" layer="1"/>
+<wire x1="37.5" y1="41.84" x2="37.5" y2="41.58" width="0.1524" layer="1"/>
+</signal>
 </signals>
